File: pmic/basic_v1/basic_v1.kicad_sch (KiCad schematic)
At the start: 69 parts, among them J1 Screw_Terminal_01x02, J2 OUTPUT, J4 Conn_01x08_Male, J5 Conn_01x08_Male, Q1 VNN7NV04, Q2 VNN7NV04, Q3 ISL9V5045S3ST, Q4 ISL9V5045S3ST, Q5 VNN7NV04, Q6 VNN7NV04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

Commit message: basic driver v1
Connections:
- net INY1: now also R4.2, U1.2 (IN)
- net INY2: now also R11.2, U5.2 (IN)
- net INY3: now also R5.2, U2.2 (IN)
- net INY4: now also R12.2, U6.2 (IN)
Changed lines of the file:
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@@
+    (effects (font (size 1.27 1.27)) (justify left bottom))
+  )
+  (label "INY3" (at 93.345 33.02 0)
     (effects (font (size 1.27 1.27)) (justify left bottom))
   )
   (label "INY1" (at 130.81 99.695 0)
+    (effects (font (size 1.27 1.27)) (justify left bottom))
+  )
+  (label "INY4" (at 93.345 66.04 0)
     (effects (font (size 1.27 1.27)) (justify left bottom))
   )
@@
   )
   (label "IGN1" (at 244.475 39.37 0)
+    (effects (font (size 1.27 1.27)) (justify left bottom))
+  )
+  (label "INY2" (at 24.13 66.04 0)
     (effects (font (size 1.27 1.27)) (justify left bottom))
   )
@@
     (effects (font (size 0.7874 0.7874)) (justify left bottom))
   )
+  (label "INY1" (at 24.13 33.02 0)
+    (effects (font (size 1.27 1.27)) (justify left bottom))
+  )
   (label "IGN2" (at 244.475 66.675 0)
