File: pmic/basic_v1/basic_v1.kicad_pcb (KiCad board)
At the start: 4 copper layers, 48 x 65.6 mm, 69 parts, among them J1 Screw_Terminal_01x02, J2 OUTPUT, J4 Conn_01x08_Male, J5 Conn_01x08_Male, Q1 VNN7NV04, Q2 VNN7NV04, Q3 ISL9V5045S3ST, Q4 ISL9V5045S3ST, Q5 VNN7NV04, Q6 VNN7NV04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

Commit message: basic driver v1
Parts:
- moved R1 41.8 mm to (164.8, 108.7)
- moved R16 37.8 mm to (207.4, 109.5), turned to 180 degrees
- moved R3 35.7 mm to (169.3, 104.3)
- moved R6 34.4 mm to (172.1, 111.4)
- moved R22 34.0 mm to (206.8, 131.6), turned to 90 degrees
- moved R4 32.2 mm to (172.7, 109.5), turned to 180 degrees
- moved R14 31.5 mm to (195.6, 109.6), turned to 180 degrees
- moved R10 31.2 mm to (200.4, 109.7)
- moved R7 29.8 mm to (180.4, 104.3)
- moved U3 29.8 mm to (172.9, 105.4), turned to 90 degrees
- moved R2 29.2 mm to (188.7, 109.7)
- moved R9 27.8 mm to (176.9, 109.3)
- moved R18 24.6 mm to (203.4, 131.6), turned to 90 degrees
- moved R15 24.3 mm to (204.1, 104.5)
- moved R13 22.7 mm to (192.3, 104.5), turned to 0 degrees
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Connections:
- R11 pad 2: Net-(R11-Pad2) -> /INY2
- R12 pad 2: Net-(R12-Pad2) -> /INY4
- R4 pad 2: Net-(R4-Pad2) -> /INY1
- R5 pad 2: Net-(R5-Pad2) -> /INY3
- U1 pad 2: Net-(R4-Pad2) -> /INY1
- U2 pad 2: Net-(R5-Pad2) -> /INY3
- U5 pad 2: Net-(R11-Pad2) -> /INY2
- U6 pad 2: Net-(R12-Pad2) -> /INY4
Routing:
- net /IGN1: track 0.00 -> 67.0 mm, vias 0 -> 2
- net VCOM: track 0.00 -> 66.0 mm, vias 0 -> 4
- net Net-(D1-Pad1): track 0.00 -> 60.8 mm, vias 0 -> 2
- net /IGN2: track 0.00 -> 58.5 mm, vias 0 -> 2
- net /ECN4: track 0.00 -> 55.6 mm
- net /IGN3: track 0.00 -> 50.9 mm, vias 0 -> 2
- net /IGN4: track 0.00 -> 50.3 mm, vias 0 -> 2
- net Net-(D4-Pad1): track 0.00 -> 49.9 mm, vias 0 -> 2
- net /INY4: track 0.00 -> 49.2 mm, vias 0 -> 2
- net Net-(D6-Pad1): track 0.00 -> 43.9 mm, vias 0 -> 2
- net /ECN3: track 0.00 -> 43.5 mm
- net +12V: track 0.00 -> 38.0 mm, vias 0 -> 7
- net +5V: track 0.00 -> 37.9 mm, vias 0 -> 1
- net /INY3: track 0.00 -> 37.0 mm, vias 0 -> 2
- net Net-(D13-Pad1): track 0.00 -> 33.4 mm, vias 0 -> 2
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- added copper zone on In2.Cu, net +12V
Other:
- board text added: "ACA E BARATO"
- board text added: "ACA ME ROMPEN EL UPITE"

Commit message: wip uefi mainboard
Parts:
- moved JP1 32.3 mm to (175.2, 117.2), turned to 90 degrees
- moved D3 18.0 mm to (203.3, 116.8)
- moved D5 18.0 mm to (197.9, 116.8)
- moved D9 18.0 mm to (199.6, 116.7)
- moved D1 18.0 mm to (196.2, 116.8)
- moved D11 18.0 mm to (206.7, 116.8)
- moved D13 18.0 mm to (201.2, 116.7)
- moved D15 18.0 mm to (208.4, 116.8)
- moved D7 18.0 mm to (205.0, 116.8)
- moved R17 18.0 mm to (196.2, 113.6)
- moved R18 18.0 mm to (203.3, 113.6)
- moved R19 18.0 mm to (197.9, 113.6)
- moved R20 18.0 mm to (205.0, 113.6)
- moved R21 18.0 mm to (199.6, 113.6)
- moved R22 18.0 mm to (206.7, 113.6)
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Routing:
- net /ECN4: track 55.6 -> 15.0 mm
- net /ECN3: track 43.5 -> 4.26 mm
- net +5V: track 37.9 -> 0.00 mm, vias 1 -> 0
- net /IGN2: track 58.5 -> 27.6 mm, vias 2 -> 1
- net /IGN1: track 67.0 -> 38.4 mm, vias 2 -> 1
- net Net-(D6-Pad1): track 43.9 -> 15.8 mm, vias 2 -> 1
- net Net-(D1-Pad1): track 60.8 -> 33.1 mm, vias 2 -> 1
- net Net-(D13-Pad1): track 33.4 -> 6.42 mm, vias 2 -> 1
- net /ECN2: track 31.5 -> 4.96 mm
- net Net-(D4-Pad1): track 49.9 -> 24.2 mm, vias 2 -> 1
- net /IGN3: track 50.9 -> 25.8 mm, vias 2 -> 1
- net /IGN4: track 50.3 -> 25.2 mm, vias 2 -> 1
- net /INY4: track 49.2 -> 27.8 mm, vias 2 -> 1
- net /INY2: track 30.2 -> 8.91 mm, vias 2 -> 1
- net /INY3: track 37.0 -> 16.0 mm, vias 2 -> 1
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Other:
- board size 48 x 65.6 mm -> 48 x 47.7 mm
- board text removed: "ACA E BARATO"
- board text removed: "ACA ME ROMPEN EL UPITE"
