File: pmic/MC33810_v1/MC33810_v1.kicad_pcb (KiCad board)
At the start: 4 copper layers, 48 x 65.6 mm, 42 parts, among them J1 Conn_01x08_Male, J2 Conn_01x08_Male, J3 Conn_01x08_Male, J4 OUTPUT, J5 Screw_Terminal_01x02, Q1 ISL9V5045S3ST, Q2 ISL9V5045S3ST, Q3 ISL9V5045S3ST, Q4 ISL9V5045S3ST, U1 MCZ33810EK

Commit message: wip uefi mainboard
Parts:
- added Churrosoft: SYM_Hot_Large, OpenEFI-STM32F_rev3:churro_new_v4, B.Cu at (133.1, 63.0)
- moved J2 20.9 mm to (131.1, 93.7)
- moved TP5 13.2 mm to (106.0, 86.8)
- moved TP6 13.2 mm to (106.0, 88.9)
- moved TP7 13.2 mm to (106.0, 91.0)
- moved TP8 13.2 mm to (106.0, 93.1)
- moved C12 13.1 mm to (114.7, 93.0)
- moved C10 12.7 mm to (127.7, 94.2)
- moved U1 12.0 mm to (122.3, 87.6)
- moved R10 11.2 mm to (130.4, 86.2)
- moved J1 10.0 mm to (142.5, 86.7)
- moved J3 9.90 mm to (101.5, 86.8)
- moved C13 9.14 mm to (114.7, 81.6)
- moved C11 8.79 mm to (128.6, 80.7)
- moved C6 5.79 mm to (135.1, 82.9)
- moved C7 5.79 mm to (142.3, 81.3)
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Connections:
- J2 pad 4: /PMIC_MAXI -> /PMIC_NOMI
- J2 pad 5: /PMIC_NOMI -> /PMIC_MAXI
Routing:
- net /FB1: track 44.3 -> 25.3 mm
- net /GD3: track 44.6 -> 29.9 mm
- net +12V: track 16.2 -> 2.47 mm, vias 0 -> 1
- net L4: track 57.4 -> 44.0 mm
- net /PMIC_ENABLE: track 17.5 -> 30.6 mm
- net /RSP: track 29.8 -> 17.6 mm
- net /FB2: track 24.4 -> 12.2 mm, vias 2 -> 0
- net M4: track 54.5 -> 42.3 mm
- net L3: track 71.2 -> 59.1 mm
- net M3: track 68.1 -> 56.2 mm
- net /FB0: track 23.7 -> 13.0 mm, vias 2 -> 0
- net /GD2: track 42.5 -> 32.1 mm
- net /FB3: track 35.1 -> 24.7 mm
- net /PMIC_NOMI: track 24.1 -> 14.1 mm, vias 1 -> 0
- net /GD0: track 26.7 -> 16.9 mm
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- added copper zone on In2.Cu, net +12V
- added copper zone on In1.Cu, net GND
Other:
- board size 48 x 65.6 mm -> 48 x 51.9 mm
