File: pmic/MC33810_v1/MC33810_v1.kicad_sch (KiCad schematic)
At the start: 42 parts, among them J1 Conn_01x08_Male, J2 Conn_01x08_Male, J3 Conn_01x08_Male, J4 OUTPUT, J5 Screw_Terminal_01x02, Q1 ISL9V5045S3ST, Q2 ISL9V5045S3ST, Q3 ISL9V5045S3ST, Q4 ISL9V5045S3ST, U1 MCZ33810EK

Commit message: wip uefi mainboard
Connections:
- net PMIC_MAXI: now also J2.5 (Pin_5); no longer J2.4 (Pin_4)
- net PMIC_NOMI: now also J2.4 (Pin_4); no longer J2.5 (Pin_5)
Changed lines of the file:
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@@
     (effects (font (size 1.27 1.27)) (justify left bottom))
   )
-  (label "PMIC_NOMI" (at 48.26 180.975 0)
+  (label "PMIC_NOMI" (at 48.26 178.435 0)
     (effects (font (size 0.7874 0.7874)) (justify left bottom))
   )
@@
     (effects (font (size 1.27 1.27)) (justify left bottom))
   )
-  (label "PMIC_MAXI" (at 48.26 178.435 0)
+  (label "PMIC_MAXI" (at 48.26 180.975 0)
     (effects (font (size 0.7874 0.7874)) (justify left bottom))
   )
