File: mainboard_uEFI/mainboard_uEFI.kicad_pcb (KiCad board)
At the start: 4 copper layers, 100 x 100 mm, 143 parts, among them J1 36638-0002, J2 Tag connect, J3 Conn_02x08_Odd_Even, J4 USB_B, J5 Conn_01x03, Q1 IRF540N, Q2 IRLZ44N, Q3 IRLZ44N, Q4 SS8050, Q5 AO3400A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

Commit message: wip uefi v4 mainboard
Parts:
- TP2, TP4, TP5, TP6: moved to B.Cu
- moved C9 85.5 mm to (189.4, 141.1)
- moved C10 85.0 mm to (211.1, 141.7), turned to 0 degrees
- moved C13 83.2 mm to (190.2, 144.0)
- moved C11 83.0 mm to (208.6, 123.0)
- moved R11 82.9 mm to (199.8, 107.4)
- moved Q7 78.0 mm to (199.6, 110.3), turned to 90 degrees
- moved R13 68.8 mm to (196.9, 110.7)
- moved J5 66.3 mm to (166.8, 121.1)
- moved C14 55.9 mm to (181.2, 118.2), turned to 90 degrees
- moved U9 54.3 mm to (175.0, 104.0), turned to 90 degrees
- moved TP2 49.6 mm to (170.5, 115.6), turned to 0 degrees
- moved C6 48.7 mm to (158.6, 130.5)
- moved R15 39.5 mm to (177.8, 97.4), turned to 90 degrees
- moved TP5 38.7 mm to (168.7, 110.1), turned to 180 degrees
- moved R14 38.7 mm to (172.8, 97.4)
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- renumbered TP| to TP8
Connections:
- U7 pad 33: +12V -> /PMIC_CS
- U8 pad 33: /AUX_OUT_1 -> /AUX_OUT_3
- U8 pad 35: /AUX_OUT_3 -> /AUX_OUT_1
- U8 pad 38: /MTR_STEP -> /MTR_FAULT
- U8 pad 39: /MTR_DIR -> /MTR_ENABLE
- U8 pad 40: /MTR_FAULT -> /MTR_STEP
- U8 pad 41: /MTR_ENABLE -> /MTR_DIR
- U8 pad 91: /AUX_IN_1 -> /AUX_IN_4
- U8 pad 92: /AUX_IN_2 -> /AUX_IN_3
- U8 pad 93: /AUX_IN_3 -> /AUX_IN_2
- U8 pad 95: /AUX_IN_4 -> /AUX_IN_1
Routing:
- net /SPI2_SCK: track 0.00 -> 110.8 mm, vias 0 -> 2
- net /SPI2_MISO: track 0.00 -> 110.8 mm, vias 0 -> 2
- net /SPI2_MOSI: track 0.00 -> 103.9 mm, vias 0 -> 2
- net /MTR_FAULT: track 0.00 -> 70.0 mm
- net CAN-: track 0.00 -> 54.9 mm, vias 0 -> 2
- net CAN+: track 0.00 -> 54.8 mm, vias 0 -> 2
- net /PMIC_CS: track 0.00 -> 49.1 mm, vias 0 -> 1
- net /MTR_ENABLE: track 29.5 -> 76.5 mm
- net /MTR_STEP: track 14.8 -> 61.1 mm
- net /MTR_DIR: track 16.4 -> 58.3 mm
- net +3V3: track 63.2 -> 102.0 mm, vias 3 -> 8
- net /PMIC_ENABLE: track 0.00 -> 38.4 mm, vias 0 -> 1
- net /AUX_OUT_1: track 0.00 -> 35.8 mm, vias 0 -> 1
- net H1: track 0.00 -> 33.8 mm
- net /AUX_OUT_2: track 0.00 -> 33.2 mm, vias 0 -> 1
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Other:
- board text added: "ACC"
- board text added: "TODO: garrar la pala"

Commit message: wip uefi mainboard, led wiring
Parts:
- moved R9 6.83 mm to (204.5, 146.1), turned to 0 degrees
- moved TP1 4.70 mm to (205.4, 140.3)
- moved C10 4.46 mm to (215.2, 143.4), turned to -90 degrees
- moved R32 4.17 mm to (226.5, 118.2)
- moved R33 3.10 mm to (226.5, 121.5), turned to 90 degrees
- moved C16 2.47 mm to (207.6, 144.8)
- moved J2 1.71 mm to (173.6, 131.6)
Connections:
- net /IN1+ renamed /IN1_P
- net /IN1- renamed /IN1_N
Routing:
- net /SYS_SWO: track 0.00 -> 42.4 mm, vias 0 -> 2
- net /LED_CAN_TX: track 0.00 -> 38.4 mm, vias 0 -> 2
- net /LED_CAN_RX: track 0.00 -> 35.8 mm, vias 0 -> 2
- net /LED2: track 0.00 -> 34.4 mm, vias 0 -> 2
- net /SYS_SWCLK: track 0.00 -> 33.9 mm, vias 0 -> 2
- net /LED1: track 0.00 -> 30.4 mm, vias 0 -> 2
- net /SYS_SWDIO: track 0.00 -> 24.5 mm, vias 0 -> 2
- net /LED0: track 0.00 -> 23.8 mm, vias 0 -> 2
- net /NRST: track 81.6 -> 89.5 mm, vias 2 -> 3
- net /CKP_VR: track 0.00 -> 6.69 mm
- net /CMP: track 0.00 -> 5.18 mm
- net /PMIC_CS: track 49.1 -> 44.4 mm
- net GND: track 13.3 -> 18.0 mm, vias 7 -> 8
- net +3V3: track 102.0 -> 105.8 mm
- net /PMIC_NOMI: track 30.4 -> 27.3 mm
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Other:
- board text removed: "TODO: garrar la pala"

Commit message: uefi v4 mainboard, wip relay
Parts:
- removed F9: 750mA, Fuse:Fuse_1206_3216Metric
- F1, F2, F3, F4, F5, F6, F7, F8: moved to B.Cu
- moved F7 34.2 mm to (222.0, 60.5), turned to -90 degrees
- moved F8 29.8 mm to (217.2, 60.5), turned to -90 degrees
- moved F5 24.9 mm to (226.8, 60.5), turned to -90 degrees
- moved F6 22.0 mm to (214.8, 60.5), turned to -90 degrees
- moved F1 9.62 mm to (210.0, 60.5), turned to -90 degrees
- moved F3 8.38 mm to (224.4, 60.5), turned to -90 degrees
- moved U11 4.86 mm to (203.5, 60.1), turned to 0 degrees
- moved U10 4.70 mm to (232.9, 60.2)
- moved H9 4.47 mm to (241.5, 59.3)
- moved F2 3.69 mm to (212.4, 60.5), turned to -90 degrees
- moved F4 0.72 mm to (219.6, 60.5), turned to -90 degrees
Connections:
- U11 pad 10: Net-(F9-Pad1) -> /PWM | Relays /R3_OUT
Routing:
- net /TIM9_CH1: track 0.00 -> 150.6 mm, vias 0 -> 2
- net /TIM9_CH2: track 0.00 -> 149.2 mm, vias 0 -> 2
- net +12V: track 119.8 -> 251.2 mm, vias 4 -> 6
- net /R_ECN_INY: track 0.00 -> 121.7 mm, vias 0 -> 2
- net /R_AAC: track 0.00 -> 121.2 mm, vias 0 -> 2
- net /R_LMB: track 0.00 -> 119.9 mm, vias 0 -> 3
- net /R_GNC_GLP: track 0.00 -> 119.6 mm, vias 0 -> 2
- net +12VA: track 20.7 -> 60.7 mm, vias 0 -> 1
- net /NRST: track 89.5 -> 52.8 mm
- net A1: track 2.68 -> 35.5 mm, vias 0 -> 1
- net Net-(F4-Pad1): track 0.00 -> 17.2 mm, vias 0 -> 1
- net /PWM | Relays /CHECK_ENGINE: track 0.00 -> 16.1 mm, vias 0 -> 1
- net Net-(F3-Pad1): track 0.00 -> 12.0 mm, vias 0 -> 1
- net D3: track 0.00 -> 11.8 mm, vias 0 -> 1
- net /PWM | Relays /MIL_OUT: track 0.00 -> 11.3 mm, vias 0 -> 1
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