File: mainboard_uEFI/mainboard_uEFI.kicad_sch (KiCad schematic)
At the start: 107 parts, among them J2 Tag connect, J3 Conn_02x08_Odd_Even, J4 USB_B, J5 Conn_01x03, Q5 AO3400A, Q6 SS8050, Q7 AO3400A, Q8 SS8050, Q9 SS8050, SW1 SW_Push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

Commit message: wip uefi v4 mainboard
Connections:
- net +12V: no longer U7.33 (SPI_CS)
- net AUX_IN_1: now also U8.95 (PB8); no longer U8.91 (PB5)
- net AUX_IN_2: now also U8.93 (PB7); no longer U8.92 (PB6)
- net AUX_IN_3: now also U8.92 (PB6); no longer U8.93 (PB7)
- net AUX_IN_4: now also U8.91 (PB5); no longer U8.95 (PB8)
- net AUX_OUT_1: now also U8.35 (PB0); no longer U8.33 (PC4)
- net AUX_OUT_3: now also U8.33 (PC4); no longer U8.35 (PB0)
- net MTR_DIR: now also U8.41 (PE10); no longer U8.39 (PE8)
- net MTR_ENABLE: now also U8.39 (PE8); no longer U8.41 (PE10)
- net MTR_FAULT: now also U8.38 (PE7); no longer U8.40 (PE9)
- net MTR_STEP: now also U8.40 (PE9); no longer U8.38 (PE7)
Changed lines of the file:
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@@
     (effects (font (size 0.889 0.889)) (justify left bottom))
   )
-  (label "AUX_IN_4" (at 246.38 130.81 0)
+  (label "AUX_IN_4" (at 246.38 123.19 0)
     (effects (font (size 0.889 0.889)) (justify left bottom))
   )
@@
     (effects (font (size 1.27 1.27)) (justify left bottom))
   )
-  (label "AUX_IN_1" (at 246.38 123.19 0)
+  (label "AUX_IN_1" (at 246.38 130.81 0)
     (effects (font (size 0.889 0.889)) (justify left bottom))
   )
@@
     (effects (font (size 0.889 0.889)) (justify left bottom))
   )
-  (label "MTR_ENABLE" (at 195.58 135.89 180)
-    (effects (font (size 0.889 0.889)) (justify right bottom))
-  )
-  (label "MTR_STEP" (at 195.58 128.27 180)
+  (label "MTR_ENABLE" (at 195.58 130.81 180)
+    (effects (font (size 0.889 0.889)) (justify right bottom))
+  )
+  (label "MTR_STEP" (at 195.58 133.35 180)
     (effects (font (size 0.889 0.889)) (justify right bottom))
   )
@@
     (effects (font (size 0.7874 0.7874)) (justify right bottom))
   )
-  (label "AUX_IN_3" (at 246.38 128.27 0)
+  (label "AUX_IN_3" (at 246.38 125.73 0)
     (effects (font (size 0.889 0.889)) (justify left bottom))
   )
@@
     (effects (font (size 0.7874 0.7874)) (justify left bottom))
   )
-  (label "MTR_FAULT" (at 195.58 133.35 180)
+  (label "MTR_FAULT" (at 195.58 128.27 180)
     (effects (font (size 0.889 0.889)) (justify right bottom))
   )
@@
     (effects (font (size 1.27 1.27)) (justify right bottom))
   )
-  (label "MTR_DIR" (at 195.58 130.81 180)
+  (label "MTR_DIR" (at 195.58 135.89 180)
     (effects (font (size 0.889 0.889)) (justify right bottom))
   )
@@
     (effects (font (size 0.889 0.889)) (justify left bottom))
   )
-  (label "AUX_OUT_3" (at 247.015 110.49 0)
+  (label "AUX_OUT_3" (at 246.38 163.83 0)
     (effects (font (size 0.889 0.889)) (justify left bottom))
   )
@@
     (effects (font (size 1.27 1.27)) (justify right bottom))
   )
-  (label "AUX_OUT_1" (at 246.38 163.83 0)
+  (label "AUX_OUT_1" (at 246.38 110.49 0)
     (effects (font (size 0.889 0.889)) (justify left bottom))
   )
@@
     (effects (font (size 0.889 0.889)) (justify right bottom))
   )
-  (label "AUX_IN_2" (at 246.38 125.73 0)
+  (label "AUX_IN_2" (at 246.38 128.27 0)
     (effects (font (size 0.889 0.889)) (justify left bottom))
   )
@@
     (pin "32")
     (pin "33")
-    (pin "33")
     (pin "34")

Commit message: wip uefi mainboard, led wiring
Connections:
- net IN1+ renamed IN1_P
- net IN1- renamed IN1_N
Changed lines of the file:
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@@
     (effects (font (size 0.889 0.889)) (justify left bottom))
   )
-  (label "IN1+" (at 325.12 100.33 180)
+  (label "IN1_P" (at 295.91 100.33 180)
     (effects (font (size 1.27 1.27)) (justify right bottom))
   )
@@
     (effects (font (size 0.9906 0.9906)) (justify left bottom))
   )
-  (label "IN1-" (at 322.58 120.65 180)
-    (effects (font (size 1.27 1.27)) (justify right bottom))
-  )
+  (label "IN1_N" (at 297.18 120.65 180)
+    (effects (font (size 1.27 1.27)) (justify right bottom))
+  )
